Commit message: Working with xacro
Signed-off-by: Patrick José Pereira <patrickelectric@gmail.com>

File: model/BlueRov2.urdf.xacro (robot description, xacro)
@@ -6,5 +6,5 @@
     <inertial>
       <mass value="11"/>
-      <inertia ixx="0" ixy="0" ixz="0" iyy="0" iyz="0" izz="0" />
+      <inertia ixx="0.1" ixy="0" ixz="0" iyy="0.1" iyz="0" izz="0.1" />
     </inertial>
     <visual>
@@ -31,3 +31,9 @@
     </plugin>
   </gazebo>
+  <buoyancy>
+      <compensation>10.3</compensation>
+      <!--origin xyz= "0 0 0"/>
+      <limit radius=".5"/>
+      <damping xyz="100 200 150" rpy="50 50 50"/-->
+  </buoyancy>
 </robot>

Commit message: Update gazebo.launch and BlueRov2.xacro
WIP: Thrusters and floating working
Is it possible to control ROV in /BlueRov2/body_command
```
import rospy
from sensor_msgs.msg import JointState

def talker():
    pub = rospy.Publisher('/BlueRov2/body_command', JointState, queue_size=10)
    rospy.init_node('joint_state_publisher')
    rate = rospy.Rate(10) # 10hz
    hello_str = JointState()
    hello_str.name = ['thr2']
    hello_str.position = [-30]
    hello_str.velocity = [-30]
    hello_str.effort = [-30]
    print(hello_str)

    while not rospy.is_shutdown():
      hello_str.header.stamp = rospy.Time.now()
      pub.publish(hello_str)
      print(hello_str)
      rate.sleep()
```

Signed-off-by: Patrick José Pereira <patrickelectric@gmail.com>

File: model/BlueRov2.urdf.xacro (robot description, xacro)
@@ -1,39 +1,121 @@
-<?xml version="1.0" encoding="UTF-8"?>
-<robot xmlns:xacro="http://www.ros.org/wiki/xacro" name="BlueRov2">
-  <link name="origin_link" />
+<?xml version="1.0"?>
+<robot name="BlueRov2" xmlns:xacro="http://www.ros.org/wiki/xacro">
+  <xacro:property name="PI" value="3.1415926535897931"/>
+  <!-- Body properties -->
+  <xacro:property name="thr12_y" value="0.115"/>
+  <xacro:property name="thr34_x" value="0.18"/>
+  <xacro:property name="thr34_y" value="0.1092"/>
+  <xacro:property name="thr5_x" value="0.17"/>
+  <xacro:property name="thr6_x" value="0.039"/>
+  <xacro:property name="thr56_z" value="0.105"/>
+  <xacro:property name="eps" value="0.00000001"/>
+  <!-- Thruster link -->
+    <xacro:macro name="thruster_dummy_link" params="name xyz rpy">
+        <joint name="${name}" type="fixed">
+            <parent link="base_link"/>
+            <child link="${name}"/>
+            <origin rpy="${rpy}" xyz="${xyz}"/>
+        </joint>
+        <link name="${name}">
+            <buoyancy><compensation>1.0</compensation></buoyancy>
+            <!--visual name="${name}">
+                <geometry>
+                    <cylinder length=".5" radius=".01"/>
+                </geometry>
+                <material name="black">
+                    <color rgba="0 0 0 1"/>
+                </material>
+            </visual>
+            <inertial>
+                <mass value=".1"/>
+                <inertia
+                    ixx=".1"
+                    ixy="0.0"
+                    ixz="0.0"
+                    iyy=".1"
+                    iyz="0.0"
+                    izz=".1"/>
+                </inertial-->
+            </link>
+            <gazebo reference="${name}">
+                <material>Gazebo/Black</material>
+            </gazebo>
+        </xacro:macro>
+  <!-- Plugin list -->
+    <gazebo>
+    <!-- Gazebo plugin listens to the body-->
+    <plugin name="freefloating_gazebo_control" filename="libfreefloating_gazebo_control.so">
+        <switchService>switch</switchService>
+        <updateRate>100</updateRate>
+        <link>base_link</link>
+        <!-- for each thruster, give the map to XYZ+RPY and the maximum effort -->
+        <thruster>
+            <effort>30</effort>
+            <name>thr1</name>
+            <map>1 0 0 0 0 ${-thr12_y}</map>
+        </thruster>
+        <thruster>
+            <effort>30</effort>
+            <name>thr2</name>
+            <map>1 0 0 0 0 ${thr12_y}</map>
+        </thruster>
+        <thruster>
+            <effort>30</effort>
+            <name>thr3</name>
+            <map>0 0 -1 ${-thr34_y} ${thr34_x} 0</map>
+        </thruster>
+        <thruster>
+            <effort>30</effort>
+            <name>thr4</name>
+            <map>0 0 -1 ${thr34_y} ${thr34_x} 0</map>
+        </thruster>
+        <thruster>
+            <effort>30</effort>
+            <name>thr5</name>
+            <map>0 0 -1 0 ${-thr5_x} 0</map>
+        </thruster>
+        <thruster>
+            <effort>30</effort>
+            <name>thr6</name>
+            <map>0 1 0 ${-thr56_z} 0 0</map>
+        </thruster>
+    </plugin>
+    </gazebo>
   <link name="base_link">
-    <!--http://docs.bluerobotics.com/brov2/#specifications-->
-    <inertial>
-      <mass value="11"/>
-      <inertia ixx="0.1" ixy="0" ixz="0" iyy="0.1" iyz="0" izz="0.1" />
-    </inertial>
     <visual>
-      <geometry>
-        <mesh filename="package://bluerov_ros_playground/model/BlueRov2.stl" scale="0.1 0.1 0.1"/>
-      </geometry>
-      <material name="base_material">
-        <color rgba="1 1 1 1" />
-      </material>
-    </visual>
-    <collision>
+      <origin xyz="0 0 0" rpy="${-PI} 0 0"/>
       <geometry>
         <mesh filename="package://bluerov_ros_playground/model/BlueRov2.stl" scale="0.1 0.1 0.1" />
       </geometry>
-    </collision>
+    </visual>
+    <inertial>
+      <origin xyz="0 0 0.0" rpy="0 0 0"/>
+      <mass value="11"/>
+    <inertia
+      ixx="5"
+      ixy="0.0"
+      ixz="0.0"
+      iyy="5"
+      iyz="5"
+      izz="5"/>
+    </inertial>
+    <!--collision>
+      <origin xyz="0 0 0" rpy="0 0 0"/>
+      <geometry>
+      <box size="0.5 0.5 0.5"/>
+      </geometry>
+    </collision-->
+    <buoyancy>
+        <compensation>1.01</compensation>
+        <origin xyz= "0 0 0"/>
+        <limit radius=".5"/>
+        <damping xyz="100 200 150" rpy="50 50 50"/>
+    </buoyancy>
   </link>
-  <joint name="base_joint" type="fixed">
-    <parent link="origin_link" />
-    <child link="base_link" />
-    <origin xyz="0 0 0" />
-  </joint>
-  <gazebo>
-    <plugin name="freefloating_gazebo_control" filename="libfreefloating_gazebo_control.so">
-    </plugin>
-  </gazebo>
-  <buoyancy>
-      <compensation>10.3</compensation>
-      <!--origin xyz= "0 0 0"/>
-      <limit radius=".5"/>
-      <damping xyz="100 200 150" rpy="50 50 50"/-->
-  </buoyancy>
+<xacro:thruster_dummy_link name="thr1" xyz="0.0 0.115 0.0" rpy="-0.0 -1.57079632679 0.0"/>
+<xacro:thruster_dummy_link name="thr2" xyz="0.0 -0.115 0.0" rpy="-0.0 -1.57079632679 0.0"/>
+<xacro:thruster_dummy_link name="thr3" xyz="0.18 0.1092 0.0" rpy="0.0 -0.0 0.0"/>
+<xacro:thruster_dummy_link name="thr4" xyz="0.18 -0.1092 0.0" rpy="0.0 -0.0 0.0"/>
+<xacro:thruster_dummy_link name="thr5" xyz="-0.17 0.0 0.0" rpy="0.0 -0.0 0.0"/>
+<xacro:thruster_dummy_link name="thr6" xyz="0.0 0.0 0.105" rpy="1.57079632679 -0.0 0.0"/>
 </robot>

Commit message: BlueRov2: Update model thrusters position
Signed-off-by: Patrick José Pereira <patrickelectric@gmail.com>

File: model/BlueRov2.urdf.xacro (robot description, xacro)
@@ -2,11 +2,4 @@
 <robot name="BlueRov2" xmlns:xacro="http://www.ros.org/wiki/xacro">
   <xacro:property name="PI" value="3.1415926535897931"/>
-  <!-- Body properties -->
-  <xacro:property name="thr12_y" value="0.115"/>
-  <xacro:property name="thr34_x" value="0.18"/>
-  <xacro:property name="thr34_y" value="0.1092"/>
-  <xacro:property name="thr5_x" value="0.17"/>
-  <xacro:property name="thr6_x" value="0.039"/>
-  <xacro:property name="thr56_z" value="0.105"/>
   <xacro:property name="eps" value="0.00000001"/>
   <!-- Thruster link -->
@@ -50,33 +43,34 @@
         <link>base_link</link>
         <!-- for each thruster, give the map to XYZ+RPY and the maximum effort -->
+        <!-- https://www.ardusub.com/images/vectored-frame.png -->
         <thruster>
             <effort>30</effort>
             <name>thr1</name>
-            <map>1 0 0 0 0 ${-thr12_y}</map>
+            <map>1 1 0 0 0 0</map>
         </thruster>
         <thruster>
             <effort>30</effort>
             <name>thr2</name>
-            <map>1 0 0 0 0 ${thr12_y}</map>
+            <map>1 -1 0 0 0 0</map>
         </thruster>
         <thruster>
             <effort>30</effort>
             <name>thr3</name>
-            <map>0 0 -1 ${-thr34_y} ${thr34_x} 0</map>
+            <map>-1 -1 0 0 0 0</map>
         </thruster>
         <thruster>
             <effort>30</effort>
             <name>thr4</name>
-            <map>0 0 -1 ${thr34_y} ${thr34_x} 0</map>
+            <map>1 -1 0 0 0 0</map>
         </thruster>
         <thruster>
             <effort>30</effort>
             <name>thr5</name>
-            <map>0 0 -1 0 ${-thr5_x} 0</map>
+            <map>0 0 0 0 0 1</map>
         </thruster>
         <thruster>
             <effort>30</effort>
             <name>thr6</name>
-            <map>0 1 0 ${-thr56_z} 0 0</map>
+            <map>0 0 0 0 0 1</map>
         </thruster>
     </plugin>
@@ -90,10 +84,10 @@
     </visual>
     <inertial>
-      <origin xyz="0 0 0.0" rpy="0 0 0"/>
+      <origin xyz="0 0 0" rpy="0 0 0"/>
       <mass value="11"/>
     <inertia
       ixx="5"
-      ixy="0.0"
-      ixz="0.0"
+      ixy="0"
+      ixz="0"
       iyy="5"
       iyz="5"
@@ -113,9 +107,11 @@
     </buoyancy>
   </link>
-<xacro:thruster_dummy_link name="thr1" xyz="0.0 0.115 0.0" rpy="-0.0 -1.57079632679 0.0"/>
-<xacro:thruster_dummy_link name="thr2" xyz="0.0 -0.115 0.0" rpy="-0.0 -1.57079632679 0.0"/>
-<xacro:thruster_dummy_link name="thr3" xyz="0.18 0.1092 0.0" rpy="0.0 -0.0 0.0"/>
-<xacro:thruster_dummy_link name="thr4" xyz="0.18 -0.1092 0.0" rpy="0.0 -0.0 0.0"/>
-<xacro:thruster_dummy_link name="thr5" xyz="-0.17 0.0 0.0" rpy="0.0 -0.0 0.0"/>
-<xacro:thruster_dummy_link name="thr6" xyz="0.0 0.0 0.105" rpy="1.57079632679 -0.0 0.0"/>
+<!-- Based on 6 thrusters vectored frame https://www.ardusub.com/images/vectored-frame.png -->
+<!-- BlueRov2 CAD https://grabcad.com/library/bluerov2-1 -->
+<xacro:thruster_dummy_link name="thr1" xyz="0.137 -0.096 0.02" rpy="0 0 0.7853981633974483"/>
+<xacro:thruster_dummy_link name="thr2" xyz="0.137 0.096 0.02" rpy="0 0 -0.7853981633974483"/>
+<xacro:thruster_dummy_link name="thr3" xyz="-0.137 -0.096 0.02" rpy="0 0 3.9269908169872414"/>
+<xacro:thruster_dummy_link name="thr4" xyz="-0.137 0.096 0.02" rpy="0 0 2.356194490192345"/>
+<xacro:thruster_dummy_link name="thr5" xyz="0 -0.111 0.07" rpy="0 1.57079632679 0"/>
+<xacro:thruster_dummy_link name="thr6" xyz="0 0.111 0.07" rpy="0 1.57079632679 0"/>
 </robot>

Commit message: BlueRov2: Update model thrusters position
Signed-off-by: Patrick José Pereira <patrickelectric@gmail.com>

File: model/BlueRov2.urdf.xacro (robot description, xacro)
@@ -2,11 +2,4 @@
 <robot name="BlueRov2" xmlns:xacro="http://www.ros.org/wiki/xacro">
   <xacro:property name="PI" value="3.1415926535897931"/>
-  <!-- Body properties -->
-  <xacro:property name="thr12_y" value="0.115"/>
-  <xacro:property name="thr34_x" value="0.18"/>
-  <xacro:property name="thr34_y" value="0.1092"/>
-  <xacro:property name="thr5_x" value="0.17"/>
-  <xacro:property name="thr6_x" value="0.039"/>
-  <xacro:property name="thr56_z" value="0.105"/>
   <xacro:property name="eps" value="0.00000001"/>
   <!-- Thruster link -->
@@ -50,33 +43,34 @@
         <link>base_link</link>
         <!-- for each thruster, give the map to XYZ+RPY and the maximum effort -->
+        <!-- https://www.ardusub.com/images/vectored-frame.png -->
         <thruster>
             <effort>30</effort>
             <name>thr1</name>
-            <map>1 0 0 0 0 ${-thr12_y}</map>
+            <map>1 1 0 0 0 0</map>
         </thruster>
         <thruster>
             <effort>30</effort>
             <name>thr2</name>
-            <map>1 0 0 0 0 ${thr12_y}</map>
+            <map>1 -1 0 0 0 0</map>
         </thruster>
         <thruster>
             <effort>30</effort>
             <name>thr3</name>
-            <map>0 0 -1 ${-thr34_y} ${thr34_x} 0</map>
+            <map>-1 -1 0 0 0 0</map>
         </thruster>
         <thruster>
             <effort>30</effort>
             <name>thr4</name>
-            <map>0 0 -1 ${thr34_y} ${thr34_x} 0</map>
+            <map>1 -1 0 0 0 0</map>
         </thruster>
         <thruster>
             <effort>30</effort>
             <name>thr5</name>
-            <map>0 0 -1 0 ${-thr5_x} 0</map>
+            <map>0 0 0 0 0 1</map>
         </thruster>
         <thruster>
             <effort>30</effort>
             <name>thr6</name>
-            <map>0 1 0 ${-thr56_z} 0 0</map>
+            <map>0 0 0 0 0 1</map>
         </thruster>
     </plugin>
@@ -113,9 +107,11 @@
     </buoyancy>
   </link>
-<xacro:thruster_dummy_link name="thr1" xyz="0.0 0.115 0.0" rpy="-0.0 -1.57079632679 0.0"/>
-<xacro:thruster_dummy_link name="thr2" xyz="0.0 -0.115 0.0" rpy="-0.0 -1.57079632679 0.0"/>
-<xacro:thruster_dummy_link name="thr3" xyz="0.18 0.1092 0.0" rpy="0.0 -0.0 0.0"/>
-<xacro:thruster_dummy_link name="thr4" xyz="0.18 -0.1092 0.0" rpy="0.0 -0.0 0.0"/>
-<xacro:thruster_dummy_link name="thr5" xyz="-0.17 0.0 0.0" rpy="0.0 -0.0 0.0"/>
-<xacro:thruster_dummy_link name="thr6" xyz="0.0 0.0 0.105" rpy="1.57079632679 -0.0 0.0"/>
+<!-- Based on 6 thrusters vectored frame https://www.ardusub.com/images/vectored-frame.png -->
+<!-- BlueRov2 CAD https://grabcad.com/library/bluerov2-1 -->
+<xacro:thruster_dummy_link name="thr1" xyz="0.137 -0.096 0.02" rpy="0.0 0.0 0.7853981633974483"/>
+<xacro:thruster_dummy_link name="thr2" xyz="0.137 0.096 0.02" rpy="0.0 0.0 -0.7853981633974483"/>
+<xacro:thruster_dummy_link name="thr3" xyz="-0.137 -0.096 0.02" rpy="0.0 0 0.0 3.9269908169872414"/>
+<xacro:thruster_dummy_link name="thr4" xyz="-0.137 0.096 0.02" rpy="0.0  0.0 2.356194490192345"/>
+<xacro:thruster_dummy_link name="thr5" xyz="0.0 -0.111 0.07" rpy="0.0 1.57079632679 0.0"/>
+<xacro:thruster_dummy_link name="thr6" xyz="0.0 0.111 0.07" rpy="0.0 1.57079632679 0.0"/>
 </robot>

Commit message: BlueRov2.urdf.xacro: Add visual back
Signed-off-by: Patrick José Pereira <patrickelectric@gmail.com>

File: model/BlueRov2.urdf.xacro (robot description, xacro)
@@ -12,5 +12,5 @@
         <link name="${name}">
             <buoyancy><compensation>1.0</compensation></buoyancy>
-            <!--visual name="${name}">
+            <visual name="${name}">
                 <geometry>
                     <cylinder length=".5" radius=".01"/>
@@ -29,5 +29,5 @@
                     iyz="0.0"
                     izz=".1"/>
-                </inertial-->
+                </inertial>
             </link>
             <gazebo reference="${name}">

Commit message: BlueRov2.urdf.xacro: Add camera
Signed-off-by: Patrick José Pereira <patrickelectric@gmail.com>

File: model/BlueRov2.urdf.xacro (robot description, xacro)
@@ -115,3 +115,61 @@
 <xacro:thruster_dummy_link name="thr5" xyz="-0.111 0 0.07" rpy="0 0 0"/>
 <xacro:thruster_dummy_link name="thr6" xyz="0.111 0 0.07" rpy="0 0 0"/>
+  <link name="camera_link">
+    <!-- visual>
+      <geometry>
+        <box size="0.1 0.1 0.1"/>
+      </geometry>
+      <material name="black">
+        <color rgba="1 1 1 1"/>
+      </material>
+    </visual -->
+  </link>
+  <joint name="camera_joint" type="fixed">
+    <parent link="base_link"/>
+    <child link="camera_link"/>
+    <origin rpy="${PI} 0 ${PI/2}" xyz="0 0.21 -0.042"/>
+    <axis xyz="1 0 0" />
+  </joint>
+  <!-- camera -->
+  <gazebo reference="camera_link">
+    <sensor type="camera" name="camera1">
+      <update_rate>30.0</update_rate>
+      <camera name="head">
+      <!-- https://elinux.com/Rpi_Camera_Module  -->
+        <horizontal_fov>1.0855</horizontal_fov>
+        <vertical_fov>0.85169</vertical_fov>
+        <image>
+          <width>1920</width>
+          <height>1080</height>
+          <format>R8G8B8</format>
+        </image>
+        <clip>
+          <near>0.01</near>
+          <far>500</far>
+        </clip>
+        <noise>
+          <type>gaussian</type>
+          <!-- Noise is sampled independently per pixel on each frame.
+               That pixel's noise value is added to each of its color
+               channels, which at that point lie in the range [0,1]. -->
+          <mean>0.0</mean>
+          <stddev>0.007</stddev>
+        </noise>
+      </camera>
+      <plugin name="camera_controller" filename="libgazebo_ros_camera.so">
+        <alwaysOn>true</alwaysOn>
+        <updateRate>0.0</updateRate>
+        <cameraName>camera</cameraName>
+        <imageTopicName>image_raw</imageTopicName>
+        <cameraInfoTopicName>camera_info</cameraInfoTopicName>
+        <frameName>camera_link</frameName>
+        <hackBaseline>0.07</hackBaseline>
+        <distortionK1>0.0</distortionK1>
+        <distortionK2>0.0</distortionK2>
+        <distortionK3>0.0</distortionK3>
+        <distortionT1>0.0</distortionT1>
+        <distortionT2>0.0</distortionT2>
+      </plugin>
+    </sensor>
+  </gazebo>
 </robot>

Commit message: finish 3D model
Signed-off-by: Patrick José Pereira <patrickelectric@gmail.com>

File: model/BlueRov2.urdf.xacro (robot description, xacro)
@@ -11,6 +11,6 @@
         </joint>
         <link name="${name}">
-            <buoyancy><compensation>1.0</compensation></buoyancy>
-            <!--visual name="${name}">
+            <!--buoyancy><compensation>1.0</compensation></buoyancy>
+            <visual name="${name}">
                 <geometry>
                     <cylinder length=".5" radius=".01"/>
@@ -19,6 +19,6 @@
                     <color rgba="0 0 0 1"/>
                 </material>
-            </visual>
-            <inertial>
+            </visual-->
+            <!--inertial>
                 <mass value=".1"/>
                 <inertia
@@ -43,34 +43,35 @@
         <link>base_link</link>
         <!-- for each thruster, give the map to XYZ+RPY and the maximum effort -->
-        <!-- https://www.ardusub.com/images/vectored-frame.png -->
+        <!-- Based on 6 thrusters vectored frame https://www.ardusub.com/images/vectored-frame.png -->
+        <!-- BlueRov2 CAD https://grabcad.com/library/bluerov2-1 -->
         <thruster>
             <effort>30</effort>
             <name>thr1</name>
-            <map>1 1 0 0 0 0</map>
+            <map>-0.707 0.707 0 0 0 -0.167</map>
         </thruster>
         <thruster>
             <effort>30</effort>
             <name>thr2</name>
-            <map>1 -1 0 0 0 0</map>
+            <map>0.707 0.707 0 0 0 0.167</map>
         </thruster>
         <thruster>
             <effort>30</effort>
             <name>thr3</name>
-            <map>-1 -1 0 0 0 0</map>
+            <map>-0.707 -0.707 0 0 0 0.167</map>
         </thruster>
         <thruster>
             <effort>30</effort>
             <name>thr4</name>
-            <map>1 -1 0 0 0 0</map>
+            <map>0.707 -0.707 0 0 0 -0.167</map>
         </thruster>
         <thruster>
             <effort>30</effort>
             <name>thr5</name>
-            <map>0 0 0 0 0 1</map>
+            <map>0 0 -1 0 -0.111 0</map>
         </thruster>
         <thruster>
             <effort>30</effort>
             <name>thr6</name>
-            <map>0 0 0 0 0 1</map>
+            <map>0 0 -1 0 0.111 0</map>
         </thruster>
     </plugin>
@@ -78,5 +79,5 @@
   <link name="base_link">
     <visual>
-      <origin xyz="0 0 0" rpy="${-PI} 0 0"/>
+      <origin xyz="0 0 0" rpy="${PI} 0 0"/>
       <geometry>
         <mesh filename="package://bluerov_ros_playground/model/BlueRov2.stl" scale="0.1 0.1 0.1" />
@@ -87,10 +88,10 @@
       <mass value="11"/>
     <inertia
-      ixx="5"
+      ixx="1"
       ixy="0"
       ixz="0"
-      iyy="5"
-      iyz="5"
-      izz="5"/>
+      iyy="1"
+      iyz="0"
+      izz="1"/>
     </inertial>
     <!--collision>
@@ -107,12 +108,4 @@
     </buoyancy>
   </link>
-<!-- Based on 6 thrusters vectored frame https://www.ardusub.com/images/vectored-frame.png -->
-<!-- BlueRov2 CAD https://grabcad.com/library/bluerov2-1 -->
-<xacro:thruster_dummy_link name="thr1" xyz="0.137 -0.096 0.02" rpy="${-PI/4} ${PI/2} 0"/>
-<xacro:thruster_dummy_link name="thr2" xyz="0.137 0.096 0.02" rpy="${PI/4} ${PI/2} 0"/>
-<xacro:thruster_dummy_link name="thr3" xyz="-0.137 -0.096 0.02" rpy="${PI/4} ${PI/2} 0"/>
-<xacro:thruster_dummy_link name="thr4" xyz="-0.137 0.096 0.02" rpy="${-PI/4} ${PI/2} 0"/>
-<xacro:thruster_dummy_link name="thr5" xyz="-0.111 0 0.07" rpy="0 0 0"/>
-<xacro:thruster_dummy_link name="thr6" xyz="0.111 0 0.07" rpy="0 0 0"/>
   <link name="camera_link">
     <!-- visual>
