Commit message: gazebo: Update 3D simulation with new freefloating
Fix #10

A better information about the model from Oliver:

The thruster map is a 6x1 vector that links a force of 1 N on the thruster
with the corresponding wrench applied to the body frame.
For example, an horizontal thruster located at 10 cm on the right side of
the body (starboard) will push along the X direction (forward) and also
induce a yaw. Its map will be : <1 0 0 0 0 0.1>

this information is redundant with the thruster link, but this link is not
mandatory and is only used for rendering. Most AUVs have fixed thrusters.
It's simpler to directly define the map instead of actual thruster links.
The links may still be used for graphical rendering, or if they are not
fixed (steering thrusters).

- Olivier Kermorgant

Signed-off-by: Patrick José Pereira <patrickelectric@gmail.com>

File: model/BlueRov2.urdf.xacro (robot description, xacro)
@@ -11,6 +11,6 @@
         </joint>
         <link name="${name}">
-            <buoyancy><compensation>1.0</compensation></buoyancy>
-            <!--visual name="${name}">
+            <!--buoyancy><compensation>1.0</compensation></buoyancy>
+            <visual name="${name}">
                 <geometry>
                     <cylinder length=".5" radius=".01"/>
@@ -19,6 +19,6 @@
                     <color rgba="0 0 0 1"/>
                 </material>
-            </visual>
-            <inertial>
+            </visual-->
+            <!--inertial>
                 <mass value=".1"/>
                 <inertia
@@ -43,34 +43,35 @@
         <link>base_link</link>
         <!-- for each thruster, give the map to XYZ+RPY and the maximum effort -->
-        <!-- https://www.ardusub.com/images/vectored-frame.png -->
+        <!-- Based on 6 thrusters vectored frame https://www.ardusub.com/images/vectored-frame.png -->
+        <!-- BlueRov2 CAD https://grabcad.com/library/bluerov2-1 -->
         <thruster>
             <effort>30</effort>
             <name>thr1</name>
-            <map>1 1 0 0 0 0</map>
+            <map>0.707 0.707 0 0 0 -0.167</map>
         </thruster>
         <thruster>
             <effort>30</effort>
             <name>thr2</name>
-            <map>1 -1 0 0 0 0</map>
+            <map>-0.707 0.707 0 0 0 0.167</map>
         </thruster>
         <thruster>
             <effort>30</effort>
             <name>thr3</name>
-            <map>-1 -1 0 0 0 0</map>
+            <map>0.707 -0.707 0 0 0 0.167</map>
         </thruster>
         <thruster>
             <effort>30</effort>
             <name>thr4</name>
-            <map>1 -1 0 0 0 0</map>
+            <map>-0.707 -0.707 0 0 0 -0.167</map>
         </thruster>
         <thruster>
             <effort>30</effort>
             <name>thr5</name>
-            <map>0 0 0 0 0 1</map>
+            <map>0 0 -1 0 -0.111 0</map>
         </thruster>
         <thruster>
             <effort>30</effort>
             <name>thr6</name>
-            <map>0 0 0 0 0 1</map>
+            <map>0 0 -1 0 0.111 0</map>
         </thruster>
     </plugin>
@@ -78,5 +79,5 @@
   <link name="base_link">
     <visual>
-      <origin xyz="0 0 0" rpy="${-PI} 0 0"/>
+      <origin xyz="0 0 0" rpy="${PI} 0 0"/>
       <geometry>
         <mesh filename="package://bluerov_ros_playground/model/BlueRov2.stl" scale="0.1 0.1 0.1" />
@@ -87,10 +88,10 @@
       <mass value="11"/>
     <inertia
-      ixx="5"
+      ixx="1"
       ixy="0"
       ixz="0"
-      iyy="5"
-      iyz="5"
-      izz="5"/>
+      iyy="1"
+      iyz="0"
+      izz="1"/>
     </inertial>
     <!--collision>
@@ -107,12 +108,4 @@
     </buoyancy>
   </link>
-<!-- Based on 6 thrusters vectored frame https://www.ardusub.com/images/vectored-frame.png -->
-<!-- BlueRov2 CAD https://grabcad.com/library/bluerov2-1 -->
-<xacro:thruster_dummy_link name="thr1" xyz="0.137 -0.096 0.02" rpy="${-PI/4} ${PI/2} 0"/>
-<xacro:thruster_dummy_link name="thr2" xyz="0.137 0.096 0.02" rpy="${PI/4} ${PI/2} 0"/>
-<xacro:thruster_dummy_link name="thr3" xyz="-0.137 -0.096 0.02" rpy="${PI/4} ${PI/2} 0"/>
-<xacro:thruster_dummy_link name="thr4" xyz="-0.137 0.096 0.02" rpy="${-PI/4} ${PI/2} 0"/>
-<xacro:thruster_dummy_link name="thr5" xyz="-0.111 0 0.07" rpy="0 0 0"/>
-<xacro:thruster_dummy_link name="thr6" xyz="0.111 0 0.07" rpy="0 0 0"/>
   <link name="camera_link">
     <!-- visual>

Commit message: BlueRov2.urdf.xacro: Add light
WIP #11

Signed-off-by: Patrick José Pereira <patrickelectric@gmail.com>

File: model/BlueRov2.urdf.xacro (robot description, xacro)
@@ -166,3 +166,31 @@
     </sensor>
   </gazebo>
+  <!-- Add light -->
+  <light type="spot" name="spot">
+    <pose>2 0 0 0 0 0</pose>
+    <diffuse>0 1 0 1</diffuse>
+    <specular>.2 .2 .2 1</specular>
+    <attenuation>
+      <range>10</range>
+      <linear>0.01</linear>
+      <constant>0.2</constant>
+      <quadratic>0.0</quadratic>
+    </attenuation>
+    <direction>0 0 -1</direction>
+    <spot>
+      <inner_angle>0.1</inner_angle>
+      <outer_angle>0.5</outer_angle>
+      <falloff>1.2</falloff>
+    </spot>
+    <cast_shadows>false</cast_shadows>
+  </light>
+  <plugin name="attach_light" filename="libAttachLightPlugin.so">
+    <link>
+      <link_name>BlueRov2::camera_link</link_name>
+      <light>
+        <pose>0 0 0.9 3.14 0 0</pose>
+        <light_name>spot</light_name>
+      </light>
+    </link>
+  </plugin>
 </robot>

Commit message: BlueRov2: Update to use .dae model
Gazebo have a better compatibility with .dae models,
now the ROV 3D model have colors

Signed-off-by: Patrick José Pereira <patrickelectric@gmail.com>

File: model/BlueRov2.urdf.xacro (robot description, xacro)
@@ -79,7 +79,7 @@
   <link name="base_link">
     <visual>
-      <origin xyz="0 0 0" rpy="${PI} 0 0"/>
+      <origin xyz="0 0 0" rpy="0 0 0"/>
       <geometry>
-        <mesh filename="package://bluerov_ros_playground/model/BlueRov2.stl" scale="0.1 0.1 0.1" />
+        <mesh filename="package://bluerov_ros_playground/model/BlueRov2.dae"/>
       </geometry>
     </visual>

Commit message: BlueRov2: Add all buoyancy foam of BlueRov2
Change from only one big foarm to multiples, like the real ROV
Fix #18

Signed-off-by: Patrick José Pereira <patrickelectric@gmail.com>

File: model/BlueRov2.urdf.xacro (robot description, xacro)
@@ -102,8 +102,18 @@
     </collision-->
     <buoyancy>
-        <compensation>1.01</compensation>
-        <origin xyz= "0 0 0"/>
-        <limit radius=".5"/>
-        <damping xyz="100 200 150" rpy="50 50 50"/>
+        <compensation>0.2525</compensation>
+        <origin xyz= "0.12585 0.111 -0.8945"/>
+    </buoyancy>
+    <buoyancy>
+        <compensation>0.2525</compensation>
+        <origin xyz= "-0.12585 0.111 -0.8945"/>
+    </buoyancy>
+    <buoyancy>
+        <compensation>0.2525</compensation>
+        <origin xyz= "-0.12585 -0.111 -0.8945"/>
+    </buoyancy>
+    <buoyancy>
+        <compensation>0.2525</compensation>
+        <origin xyz= "0.12585 -0.111 -0.8945"/>
     </buoyancy>
   </link>

Commit message: BlueRov2.urdf.xacro: Update camera position
Signed-off-by: Patrick José Pereira <patrickelectric@gmail.com>

File: model/BlueRov2.urdf.xacro (robot description, xacro)
@@ -131,5 +131,5 @@
     <parent link="base_link"/>
     <child link="camera_link"/>
-    <origin rpy="${PI} 0 ${PI/2}" xyz="0 0.21 -0.042"/>
+    <origin rpy="${PI} 0 ${PI/2}" xyz="0 0.21 -0.067"/>
     <axis xyz="1 0 0" />
   </joint>
